File: ultrafalcon.kicad_sch (KiCad schematic)
At the start: 1 part, among them SW1 RotaryEncoder

Commit message: jan17 updates
Parts:
- added C1, C2: 0.01uF, ct-kicad:C0402, symbol ct-kicad:CL05B104KO5NNNC
- added C3: 1uF, ct-kicad:C0402, symbol ct-kicad:CL05B104KO5NNNC
- added H1, H2: MountingHole, MountingHole:MountingHole_3.2mm_M3_Pad_Via, symbol Mechanical:MountingHole
- added J1: Conn_01x08_Socket, Connector_JST:JST_EH_B8B-EH-A_1x08_P2.50mm_Vertical, symbol Connector:Conn_01x08_Socket
- added R1: 330, ct-kicad:R0603, symbol ct-kicad:0603WAF3300T5E
- added R2, R3, R4, R5: 10k, ct-kicad:R0603, symbol ct-kicad:0603WAF3300T5E
- added U1, U10, U11, U12, U13, U14, U15, U16, U17, U18, U2, U3, U4, U5, U6, U7, U8, U9: SK6812MINI-E_C5149201, ct-kicad:YS-SK6812MINI-E-casuanoob, symbol ct-kicad:SK6812MINI-E_C5149201
- SW1: footprint fingerpunch:PERS56v3 -> ct-kicad:PER60
Connections:
- net at SW1.A: now also C2.1, R2.1, R4.1
- net at SW1.B: now also C1.1, R3.1, R5.1
- net GND: now reaches SW1.C
- net GND: now also C1.2, C2.2, C3.2, J1.1 (Pin_1), U1.3 (GND), U10.3 (GND), U11.3 (GND), U12.3 (GND), U13.3 (GND), U14.3 (GND), U15.3 (GND), U16.3 (GND), U17.3 (GND), U18.3 (GND), U2.3 (GND), U3.3 (GND), U4.3 (GND), U5.3 (GND), U6.3 (GND), U7.3 (GND), U8.3 (GND), U9.3 (GND)
- new net: U15.2 (DOUT), U16.4 (DIN)
- new net: U14.2 (DOUT), U15.4 (DIN)
- new net: U13.4 (DIN), U6.2 (DOUT)
- new net: U5.2 (DOUT), U6.4 (DIN)
- new net: U11.2 (DOUT), U12.4 (DIN)
- new net: U10.2 (DOUT), U11.4 (DIN)
- new net: R1.2, U7.4 (DIN)
- new net: U4.2 (DOUT), U5.4 (DIN)
- new net: U3.2 (DOUT), U4.4 (DIN)
- new net: U16.2 (DOUT), U17.4 (DIN)
- new net: U2.2 (DOUT), U3.4 (DIN)
- new net: U17.2 (DOUT), U18.4 (DIN)
- new net: U8.2 (DOUT), U9.4 (DIN)
- new net: U7.2 (DOUT), U8.4 (DIN)
- new net: U10.4 (DIN), U9.2 (DOUT)
- new net: U13.2 (DOUT), U14.4 (DIN)
- new net: U1.4 (DIN), U12.2 (DOUT)
- new net: U1.2 (DOUT), U2.4 (DIN)
- new net ENCODER_A: J1.3 (Pin_3), R4.2
- new net ENCODER_B: J1.4 (Pin_4), R5.2
- new net LED_DI: J1.5 (Pin_5), R1.1
- new net LED_DO: J1.6 (Pin_6), U18.2 (DOUT)
- new net SWITCH_A: J1.7 (Pin_7)
- new net SWITCH_B: J1.8 (Pin_8)
- new net VCC: C3.1, J1.2 (Pin_2), R2.2, R3.2, U1.1 (VDD), U10.1 (VDD), U11.1 (VDD), U12.1 (VDD), U13.1 (VDD), U14.1 (VDD), U15.1 (VDD), U16.1 (VDD), U17.1 (VDD), U18.1 (VDD), U2.1 (VDD), U3.1 (VDD), U4.1 (VDD), U5.1 (VDD), U6.1 (VDD), U7.1 (VDD), U8.1 (VDD), U9.1 (VDD)
Other:
- moved on the sheet: SW1

Commit message: v5
Parts:
- removed U13, U14, U15, U16, U17, U18: SK6812MINI-E_C5149201, ct-kicad:YS-SK6812MINI-E-casuanoob, symbol ct-kicad:SK6812MINI-E_C5149201
- added SW2: SW_Push, ct-kicad:SW_MX_cutout, symbol Switch:SW_Push
- added U1, U19, U2, U20, U21, U22, U23, U24, U25, U26, U27, U28, U29, U3, U30, U4, U5, U6: SK6805-EC15, ct-kicad:LED-SMD_4P-L1.5-W1.5-BL, symbol ct-kicad:SK6805-EC15
- C1, C2: value 0.01uF -> CL05B104KO5NNNC
- C3: value 1uF -> CL05B104KO5NNNC
- R1: value 330 -> 0603WAF3300T5E
- R2, R3, R4, R5: value 10k -> 0603WAF3300T5E
- U10, U11, U12, U7, U8, U9: value SK6812MINI-E_C5149201 -> SK6805-EC15; footprint ct-kicad:YS-SK6812MINI-E-casuanoob -> ct-kicad:LED-SMD_4P-L1.5-W1.5-BL; symbol ct-kicad:SK6812MINI-E_C5149201 -> ct-kicad:SK6805-EC15; LCSC C5149201 -> C2890035
- U13: renamed from U1; value SK6812MINI-E_C5149201 -> SK6805-EC15; footprint ct-kicad:YS-SK6812MINI-E-casuanoob -> ct-kicad:LED-SMD_4P-L1.5-W1.5-BL; symbol ct-kicad:SK6812MINI-E_C5149201 -> ct-kicad:SK6805-EC15; LCSC C5149201 -> C2890035
- U14: renamed from U2; value SK6812MINI-E_C5149201 -> SK6805-EC15; footprint ct-kicad:YS-SK6812MINI-E-casuanoob -> ct-kicad:LED-SMD_4P-L1.5-W1.5-BL; symbol ct-kicad:SK6812MINI-E_C5149201 -> ct-kicad:SK6805-EC15; LCSC C5149201 -> C2890035
- U15: renamed from U3; value SK6812MINI-E_C5149201 -> SK6805-EC15; footprint ct-kicad:YS-SK6812MINI-E-casuanoob -> ct-kicad:LED-SMD_4P-L1.5-W1.5-BL; symbol ct-kicad:SK6812MINI-E_C5149201 -> ct-kicad:SK6805-EC15; LCSC C5149201 -> C2890035
- U16: renamed from U4; value SK6812MINI-E_C5149201 -> SK6805-EC15; footprint ct-kicad:YS-SK6812MINI-E-casuanoob -> ct-kicad:LED-SMD_4P-L1.5-W1.5-BL; symbol ct-kicad:SK6812MINI-E_C5149201 -> ct-kicad:SK6805-EC15; LCSC C5149201 -> C2890035
- U17: renamed from U5; value SK6812MINI-E_C5149201 -> SK6805-EC15; footprint ct-kicad:YS-SK6812MINI-E-casuanoob -> ct-kicad:LED-SMD_4P-L1.5-W1.5-BL; symbol ct-kicad:SK6812MINI-E_C5149201 -> ct-kicad:SK6805-EC15; LCSC C5149201 -> C2890035
- U18: renamed from U6; value SK6812MINI-E_C5149201 -> SK6805-EC15; footprint ct-kicad:YS-SK6812MINI-E-casuanoob -> ct-kicad:LED-SMD_4P-L1.5-W1.5-BL; symbol ct-kicad:SK6812MINI-E_C5149201 -> ct-kicad:SK6805-EC15; LCSC C5149201 -> C2890035
Connections:
- net GND: now also U10.1 (VDD), U11.1 (VDD), U12.1 (VDD), U13.1 (VDD), U14.1 (VDD), U15.1 (VDD), U16.1 (VDD), U17.1 (VDD), U18.1 (VDD), U7.1 (VDD), U8.1 (VDD), U9.1 (VDD), U1.1 (VDD), U19.1 (VDD), U2.1 (VDD), U20.1 (VDD), U21.1 (VDD), U22.1 (VDD), U23.1 (VDD), U24.1 (VDD), U25.1 (VDD), U26.1 (VDD), U27.1 (VDD), U28.1 (VDD), U29.1 (VDD), U3.1 (VDD), U30.1 (VDD), U4.1 (VDD), U5.1 (VDD), U6.1 (VDD); no longer U10.3 (GND), U11.3 (GND), U12.3 (GND), U13.3 (GND), U14.3 (GND), U15.3 (GND), U16.3 (GND), U17.3 (GND), U18.3 (GND), U7.3 (GND), U8.3 (GND), U9.3 (GND)
- net LED_DO: now also U30.3 (DOUT)
- net VCC: now also U10.4 (GND), U11.4 (GND), U12.4 (GND), U13.4 (GND), U14.4 (GND), U15.4 (GND), U16.4 (GND), U17.4 (GND), U18.4 (GND), U7.4 (GND), U8.4 (GND), U9.4 (GND), U1.4 (GND), U19.4 (GND), U2.4 (GND), U20.4 (GND), U21.4 (GND), U22.4 (GND), U23.4 (GND), U24.4 (GND), U25.4 (GND), U26.4 (GND), U27.4 (GND), U28.4 (GND), U29.4 (GND), U3.4 (GND), U30.4 (GND), U4.4 (GND), U5.4 (GND), U6.4 (GND); no longer U10.1 (VDD), U11.1 (VDD), U12.1 (VDD), U13.1 (VDD), U14.1 (VDD), U15.1 (VDD), U16.1 (VDD), U17.1 (VDD), U18.1 (VDD), U7.1 (VDD), U8.1 (VDD), U9.1 (VDD)
- net at U18.2 (DIN): now also U17.3 (DOUT)
- net at U17.2 (DIN): now also U16.3 (DOUT); no longer U18.4 (DIN)
- net at U11.2 (DIN): now also U10.3 (DOUT); no longer U12.4 (DIN)
- net at U10.2 (DIN): now also U9.3 (DOUT); no longer U11.4 (DIN)
- net at R1.2: now also U1.2 (DIN); no longer U7.4 (DIN)
- net at U16.2 (DIN): now also U15.3 (DOUT); no longer U17.4 (DIN)
- net at U15.2 (DIN): now also U14.3 (DOUT); no longer U16.4 (DIN)
- net at U14.2 (DIN): now also U13.3 (DOUT); no longer U15.4 (DIN)
- net at U8.2 (DIN): now also U7.3 (DOUT); no longer U9.4 (DIN)
- net LED_TO_OUTER_CHAIN: now reaches U7.2 (DIN)
- net LED_TO_OUTER_CHAIN: now also U6.3 (DOUT); no longer U8.4 (DIN)
- net at U9.2 (DIN): now also U8.3 (DOUT); no longer U10.4 (DIN)
- net at U12.2 (DIN): now also U11.3 (DOUT); no longer U13.4 (DIN)
- net at U13.2 (DIN): now also U12.3 (DOUT); no longer U14.4 (DIN)
- new net: U18.3 (DOUT), U19.2 (DIN)
- new net: U2.3 (DOUT), U3.2 (DIN)
- new net: U3.3 (DOUT), U4.2 (DIN)
- new net: U26.3 (DOUT), U27.2 (DIN)
- new net: U27.3 (DOUT), U28.2 (DIN)
- new net: U25.3 (DOUT), U26.2 (DIN)
- new net: U4.3 (DOUT), U5.2 (DIN)
- new net: U5.3 (DOUT), U6.2 (DIN)
- new net: U1.3 (DOUT), U2.2 (DIN)
- new net: U23.3 (DOUT), U24.2 (DIN)
- new net: U24.3 (DOUT), U25.2 (DIN)
- new net: U19.3 (DOUT), U20.2 (DIN)
- new net: U29.3 (DOUT), U30.2 (DIN)
- new net: U22.3 (DOUT), U23.2 (DIN)
- new net: U21.3 (DOUT), U22.2 (DIN)
- new net: U28.3 (DOUT), U29.2 (DIN)
- new net: U20.3 (DOUT), U21.2 (DIN)
- no-connect marks 0 -> 2
Other:
- moved on the sheet: R1, U15, U16, U17, U18
